Commit message: Update pibo.urdf

File: data/pibo/pibo.urdf (robot description, URDF)
Before this commit: robot pibo_10dof, 11 links, 10 joints
Joints:
- joint ankle_l_joint: axis -1 0 0 -> 0 1 0; limit lower=-0.4363 upper=0.4363 effort=1.0 velocity=1.0 -> lower=-0.4363 upper=0.4363 effort=1.0 velocity=2.0; origin xyz=0 0 -0.110 -> xyz=0.00257 -0.00583 -0.07298
- joint ankle_r_joint: axis -1 0 0 -> 0 1 0; limit lower=-0.4363 upper=0.4363 effort=1.0 velocity=1.0 -> lower=-0.4363 upper=0.4363 effort=1.0 velocity=2.0; origin xyz=0 0 -0.110 -> xyz=-0.00230 -0.00733 -0.07272
- joint elbow_l_joint: axis -1 0 0 -> 0 1 0; limit lower=-0.5236 upper=0.5236 effort=1.0 velocity=1.0 -> lower=-0.5236 upper=0.5236 effort=1.0 velocity=2.0; origin xyz=0 0.050 -0.040 -> xyz=0.03852 0.00008 -0.02552
- joint elbow_r_joint: axis -1 0 0 -> 0 1 0; limit lower=-0.5236 upper=0.5236 effort=1.0 velocity=1.0 -> lower=-0.5236 upper=0.5236 effort=1.0 velocity=2.0; origin xyz=0 -0.050 -0.040 -> xyz=-0.03849 -0.00069 -0.02580
- joint head_pan_joint: limit lower=-0.8727 upper=0.8727 effort=1.0 velocity=1.0 -> lower=-0.8727 upper=0.8727 effort=1.0 velocity=2.0; origin xyz=0 0 0.125 -> xyz=0.00000 0.00007 0.23833
- joint head_tilt_joint: axis 0 1 0 -> 1 0 0; limit lower=-0.4363 upper=0.4363 effort=1.0 velocity=1.0 -> lower=-0.4363 upper=0.4363 effort=1.0 velocity=2.0; origin xyz=0 0 0.040 -> xyz=0.00066 0.00007 0.04793
- joint hip_l_joint: limit lower=-0.6109 upper=0.6109 effort=1.0 velocity=1.0 -> lower=-0.6109 upper=0.6109 effort=1.0 velocity=2.0; origin xyz=0 0.035 -0.005 -> xyz=0.03301 0.00024 0.11176
- joint hip_r_joint: limit lower=-0.6109 upper=0.6109 effort=1.0 velocity=1.0 -> lower=-0.6109 upper=0.6109 effort=1.0 velocity=2.0; origin xyz=0 -0.035 -0.005 -> xyz=-0.03328 0.00202 0.11180
- joint shoulder_l_joint: axis 0 1 0 -> 1 0 0; limit lower=-1.3963 upper=1.3963 effort=1.0 velocity=1.0 -> lower=-1.3963 upper=1.3963 effort=1.0 velocity=2.0; origin xyz=0 0.065 0.085 rpy=0 -1.5708 0 -> xyz=0.06451 0.00014 0.20270
- joint shoulder_r_joint: axis 0 -1 0 -> -1 0 0; limit lower=-1.3963 upper=1.3963 effort=1.0 velocity=1.0 -> lower=-1.3963 upper=1.3963 effort=1.0 velocity=2.0; origin xyz=0 -0.065 0.085 rpy=0 -1.5708 0 -> xyz=-0.06446 0.00014 0.20304
